File: rc-256page.kicad_pcb (KiCad board)
At the start: 2 copper layers, 99.1 x 49.9 mm, 13 parts, among them J1 RC2014, U1 SST39SF010, U2 AS6C1008, U3 74HCT138, U4 74HCT174, U5 74HCT257

Commit message: Minor layout tweaks
Routing:
- net +5V: track 141.8 -> 160.3 mm
- net A11: track 64.0 -> 57.3 mm
- net A7: track 90.8 -> 92.8 mm, vias 2 -> 1
- net MEM_A15: track 71.4 -> 69.7 mm, vias 2 -> 1
- net A5: track 82.4 -> 81.0 mm
- net A4: track 77.2 -> 75.8 mm
- net ~WR: track 105.5 -> 105.0 mm, vias 4 -> 3
- net A6: track 93.5 -> 93.0 mm
- net ~MREQ: vias 3 -> 2
